File: Hardware/Lightbox2.sch (EAGLE design)
At the start: 12 parts, among them IC1 7805T, U1 328P, Y1 16MHz

Commit message: Schematic and PCB design for final review
Parts:
- removed JP2: (no value), pinhead:PINHD-1X2
- removed R1: 10k, SparkFun-Resistors:10KOHM-0603-1/10W-1%
- added BATTERY, SWITCH: (no value), pinhead:PINHD-1X2
- added R2: (no value), adafruit:R-US_0204/5
- renumbered JP1 to PULSESENSOR, JP3 to LCD
Connections:
- net 9V: now also BATTERY.2, SWITCH.1, SWITCH.2; no longer JP2.2
- net GND: now also BATTERY.1; no longer JP2.1
- net PD3: now also R2.2; no longer R1.2
- net VCC: now also R2.1; no longer R1.1
Changed lines of the file:
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@@
 <part name="U1" library="SparkFun-IC-Microcontroller" library_urn="urn:adsk.eagle:library:525" deviceset="ATMEGA328P_PDIP" device="" package3d_urn="urn:adsk.eagle:package:38942/1" value="328P"/>
 <part name="LED1" library="adafruit" library_urn="urn:adsk.eagle:library:420" deviceset="LED" device="5MM" package3d_urn="urn:adsk.eagle:package:6240538/1"/>
-<part name="JP1" library="adafruit" library_urn="urn:adsk.eagle:library:420" deviceset="PINHD-1X3" device="" package3d_urn="urn:adsk.eagle:package:6240710/1"/>
-<part name="JP3" library="pinhead" library_urn="urn:adsk.eagle:library:325" deviceset="PINHD-1X4" device="" package3d_urn="urn:adsk.eagle:package:22407/2"/>
+<part name="PULSESENSOR" library="adafruit" library_urn="urn:adsk.eagle:library:420" deviceset="PINHD-1X3" device="" package3d_urn="urn:adsk.eagle:package:6240710/1"/>
+<part name="LCD" library="pinhead" library_urn="urn:adsk.eagle:library:325" deviceset="PINHD-1X4" device="" package3d_urn="urn:adsk.eagle:package:22407/2"/>
 <part name="C1" library="adafruit" library_urn="urn:adsk.eagle:library:420" deviceset="C-US" device="025-024X044" package3d_urn="urn:adsk.eagle:package:6240324/1" value="22pF"/>
 <part name="C2" library="adafruit" library_urn="urn:adsk.eagle:library:420" deviceset="C-US" device="025-024X044" package3d_urn="urn:adsk.eagle:package:6240324/1" value="22pF"/>
@@
 <part name="P+1" library="supply1" library_urn="urn:adsk.eagle:library:371" deviceset="VCC" device=""/>
 <part name="Y1" library="SparkFun-Clocks" library_urn="urn:adsk.eagle:library:511" deviceset="CRYSTAL-16MHZ" device="PTH-HC49US" package3d_urn="urn:adsk.eagle:package:37515/1" value="16MHz"/>
-<part name="R1" library="SparkFun-Resistors" library_urn="urn:adsk.eagle:library:532" deviceset="10KOHM" device="-0603-1/10W-1%" package3d_urn="urn:adsk.eagle:package:39650/1" value="10k"/>
-<part name="JP2" library="pinhead" library_urn="urn:adsk.eagle:library:325" deviceset="PINHD-1X2" device="" package3d_urn="urn:adsk.eagle:package:22435/2"/>
+<part name="BATTERY" library="pinhead" library_urn="urn:adsk.eagle:library:325" deviceset="PINHD-1X2" device="" package3d_urn="urn:adsk.eagle:package:22435/2"/>
+<part name="SWITCH" library="pinhead" library_urn="urn:adsk.eagle:library:325" deviceset="PINHD-1X2" device="" package3d_urn="urn:adsk.eagle:package:22435/2"/>
+<part name="R2" library="adafruit" library_urn="urn:adsk.eagle:library:420" deviceset="R-US_" device="0204/5" package3d_urn="urn:adsk.eagle:package:6240595/1"/>
 </parts>
 <sheets>
@@
 <attribute name="VALUE" x="108.712" y="71.755" size="1.778" layer="96" rot="R180"/>
 </instance>
-<instance part="JP1" gate="A" x="15.24" y="88.9" rot="R270">
+<instance part="PULSESENSOR" gate="A" x="15.24" y="88.9" rot="R270">
 <attribute name="NAME" x="20.955" y="95.25" size="1.778" layer="95" rot="R270"/>
 <attribute name="VALUE" x="7.62" y="95.25" size="1.778" layer="96" rot="R270"/>
 </instance>
-<instance part="JP3" gate="A" x="101.6" y="86.36">
+<instance part="LCD" gate="A" x="101.6" y="86.36">
 <attribute name="NAME" x="95.25" y="94.615" size="1.778" layer="95"/>
 <attribute name="VALUE" x="95.25" y="78.74" size="1.778" layer="96"/>
@@
 <attribute name="VALUE" x="20.828" y="50.8" size="1.778" layer="96" font="vector" rot="R270" align="top-center"/>
 </instance>
-<instance part="R1" gate="G$1" x="88.9" y="45.72" rot="R90">
-<attribute name="NAME" x="87.376" y="45.72" size="1.778" layer="95" font="vector" rot="R90" align="bottom-center"/>
-<attribute name="VALUE" x="90.424" y="45.72" size="1.778" layer="96" font="vector" rot="R90" align="top-center"/>
-</instance>
-<instance part="JP2" gate="G$1" x="-10.16" y="40.64" rot="R180">
-<attribute name="NAME" x="-3.81" y="34.925" size="1.778" layer="95" rot="R180"/>
-<attribute name="VALUE" x="-3.81" y="45.72" size="1.778" layer="96" rot="R180"/>
+<instance part="BATTERY" gate="G$1" x="-10.16" y="30.48" rot="R180">
+<attribute name="NAME" x="-3.81" y="24.765" size="1.778" layer="95" rot="R180"/>
+<attribute name="VALUE" x="-3.81" y="35.56" size="1.778" layer="96" rot="R180"/>
+</instance>
+<instance part="SWITCH" gate="G$1" x="-10.16" y="45.72" rot="R180">
+<attribute name="NAME" x="-3.81" y="40.005" size="1.778" layer="95" rot="R180"/>
+<attribute name="VALUE" x="-3.81" y="50.8" size="1.778" layer="96" rot="R180"/>
+</instance>
+<instance part="R2" gate="G$1" x="88.9" y="45.72" rot="R90">
+<attribute name="NAME" x="87.4014" y="44.45" size="1.778" layer="95" rot="R90"/>
+<attribute name="VALUE" x="92.202" y="41.91" size="1.778" layer="96" rot="R90"/>
 </instance>
 </instances>
@@
 </segment>
 <segment>
-<pinref part="JP1" gate="A" pin="3"/>
+<pinref part="PULSESENSOR" gate="A" pin="3"/>
 <wire x1="12.7" y1="91.44" x2="2.54" y2="91.44" width="0.1524" layer="91"/>
 <pinref part="GND5" gate="1" pin="GND"/>
 </segment>
 <segment>
-<pinref part="JP3" gate="A" pin="2"/>
+<pinref part="LCD" gate="A" pin="2"/>
 <wire x1="99.06" y1="88.9" x2="114.3" y2="88.9" width="0.1524" layer="91"/>
 <pinref part="GND6" gate="1" pin="GND"/>
@@
 <label x="7.62" y="25.4" size="1.778" layer="95"/>
 <wire x1="-7.62" y1="25.4" x2="30.48" y2="25.4" width="0.1524" layer="91"/>
-<pinref part="JP2" gate="G$1" pin="1"/>
-<wire x1="-7.62" y1="25.4" x2="-7.62" y2="38.1" width="0.1524" layer="91"/>
+<pinref part="BATTERY" gate="G$1" pin="1"/>
+<wire x1="-7.62" y1="25.4" x2="-7.62" y2="27.94" width="0.1524" layer="91"/>
 </segment>
 <segment>
@@
 <pinref part="P+1" gate="VCC" pin="VCC"/>
 <wire x1="88.9" y1="33.02" x2="88.9" y2="40.64" width="0.1524" layer="91"/>
-<pinref part="R1" gate="G$1" pin="1"/>
+<pinref part="R2" gate="G$1" pin="1"/>
 <wire x1="88.9" y1="40.64" x2="88.9" y2="43.18" width="0.1524" layer="91"/>
 <junction x="88.9" y="40.64"/>
@@
 <wire x1="22.86" y1="71.12" x2="15.24" y2="71.12" width="0.1524" layer="91"/>
 <wire x1="15.24" y1="71.12" x2="-7.62" y2="81.28" width="0.1524" layer="91"/>
-<pinref part="JP1" gate="A" pin="2"/>
+<pinref part="PULSESENSOR" gate="A" pin="2"/>
 <wire x1="15.24" y1="71.12" x2="15.24" y2="91.44" width="0.1524" layer="91"/>
 <junction x="15.24" y="71.12"/>
-<pinref part="JP3" gate="A" pin="1"/>
+<pinref part="LCD" gate="A" pin="1"/>
 <wire x1="99.06" y1="91.44" x2="22.86" y2="91.44" width="0.1524" layer="91"/>
 <wire x1="22.86" y1="91.44" x2="22.86" y2="71.12" width="0.1524" layer="91"/>
@@
 <wire x1="-7.62" y1="73.66" x2="-7.62" y2="81.28" width="0.1524" layer="91"/>
 <label x="25.4" y="71.12" size="1.778" layer="95"/>
+<label x="-15.24" y="78.74" size="1.778" layer="95"/>
 </segment>
 </net>
@@
 <wire x1="78.74" y1="48.26" x2="86.36" y2="48.26" width="0.1524" layer="91"/>
 <wire x1="86.36" y1="48.26" x2="86.36" y2="53.34" width="0.1524" layer="91"/>
-<pinref part="R1" gate="G$1" pin="2"/>
 <wire x1="88.9" y1="50.8" x2="88.9" y2="53.34" width="0.1524" layer="91"/>
 <junction x="88.9" y="53.34"/>
+<pinref part="R2" gate="G$1" pin="2"/>
 </segment>
 </net>
 <net name="PC0/ADC0" class="0">
 <segment>
-<pinref part="JP1" gate="A" pin="1"/>
+<pinref part="PULSESENSOR" gate="A" pin="1"/>
 <wire x1="17.78" y1="96.52" x2="17.78" y2="91.44" width="0.1524" layer="91"/>
 <pinref part="U1" gate="G$1" pin="PC0(ADC0)"/>
@@
 <wire x1="78.74" y1="68.58" x2="81.28" y2="68.58" width="0.1524" layer="91"/>
 <wire x1="81.28" y1="68.58" x2="81.28" y2="86.36" width="0.1524" layer="91"/>
-<pinref part="JP3" gate="A" pin="3"/>
+<pinref part="LCD" gate="A" pin="3"/>
 <wire x1="81.28" y1="86.36" x2="99.06" y2="86.36" width="0.1524" layer="91"/>
 </segment>
@@
 <wire x1="78.74" y1="66.04" x2="83.82" y2="66.04" width="0.1524" layer="91"/>
 <wire x1="83.82" y1="66.04" x2="83.82" y2="83.82" width="0.1524" layer="91"/>
-<pinref part="JP3" gate="A" pin="4"/>
+<pinref part="LCD" gate="A" pin="4"/>
 <wire x1="83.82" y1="83.82" x2="99.06" y2="83.82" width="0.1524" layer="91"/>
 </segment>
@@
 <net name="9V" class="0">
 <segment>
-<pinref part="JP2" gate="G$1" pin="2"/>
+<pinref part="BATTERY" gate="G$1" pin="2"/>
+<wire x1="-7.62" y1="30.48" x2="-7.62" y2="43.18" width="0.1524" layer="91"/>
+<pinref part="SWITCH" gate="G$1" pin="1"/>
+<label x="-10.16" y="33.02" size="1.778" layer="95"/>
+</segment>
+<segment>
 <pinref part="IC1" gate="A1" pin="VI"/>
-<wire x1="-7.62" y1="40.64" x2="-7.62" y2="53.34" width="0.1524" layer="91"/>
+<wire x1="-7.62" y1="45.72" x2="-7.62" y2="53.34" width="0.1524" layer="91"/>
 <label x="-12.7" y="48.26" size="1.778" layer="95"/>
-</segment>
-</net>
+<pinref part="SWITCH" gate="G$1" pin="2"/>
+</segment>
+</net>
