File: Hardware/PCBwGND.brd (EAGLE design)
At the start: 45.7 x 58.1 mm, 18 parts, among them IC1 7805T, U1 328P, Y1 16MHz

Commit message: Add ground plane to reduce photoetching area
Parts:
- moved 10UF_2 5.39 mm to (12.7, 24.1)
- moved BATTERY 5.39 mm to (34.3, 39.4)
- moved PULSESENSOR 5.39 mm to (34.3, 31.8)
- moved U1 5.39 mm to (25.4, 22.9)
- moved C2 5.39 mm to (5.08, 10.2)
- moved IC1 5.39 mm to (7.62, 41.9)
- moved LCD 5.39 mm to (34.3, 21.6)
- moved LED1 5.39 mm to (6.35, 24.1)
- moved LED2 5.39 mm to (31.8, 3.81)
- moved R1 5.39 mm to (34.3, 10.2)
- moved R4 5.39 mm to (15.2, 10.2)
- moved SW1 5.39 mm to (14.0, 15.2)
- moved SWITCH 5.39 mm to (16.5, 39.4)
- moved Y1 5.39 mm to (12.7, 5.08)
- moved 10UF_1 5.39 mm to (15.2, 30.5)
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Routing:
- net GND: track 118.9 -> 0.00 mm
- net PD3: track 19.4 -> 18.3 mm
- added copper zone on layer 1, net GND
- added copper zone on layer 16, net GND
Other:
- board size 45.7 x 58.1 mm -> 39.4 x 54.3 mm
